Commit message: mo hinh xe: thay so dat tam bang kich thuoc do that
URDF cu mo ta mot chiec xe duong kinh 1 m (chassis ban kinh 0.5, hai banh cach
nhau 1.1 m) - khong dinh gi den xe that. Kich thuoc do bang thuoc:

  hai banh sau cach nhau   200 mm
  truc banh sau            lui 14 mm sau tam
  banh da huong truoc      tien 35 mm truoc tam
  duong kinh banh sau      64.5 mm
  duong kinh than xe       181.40 mm

robot.urdf.xacro viet lai theo tham so xacro, moi hinh hoc va moment quan tinh
deu suy ra tu cac so tren. Tach rieng hai nhom: nhom DA DO va nhom CHUA DO
(be day than, be rong lop, ban kinh bi, chieu cao LiDAR/IMU, khoi luong) de
sau nay do duoc thi biet sua o dau.

Ba cho khac phai khop theo, neu khong dong hoc se sai:
  gazebo_control.xacro  wheel_separation 1.1 -> 0.200, wheel_radius 0.05 -> 0.03225
  firmware              WHEEL_SEPARATION_M 0.190 -> 0.200, WHEEL_RADIUS_M -> 0.03225
  navigation.yaml       robot_radius 0.6 -> 0.13, inflation_radius 0.75 -> 0.25

robot_radius khong lay ban kinh than (0.0907) ma lay goc ngoai banh sau, vi
banh nho ra ngoai than: sqrt(0.046^2 + 0.113^2) = 0.122 m, lam tron 0.13.
Giu 0.75 cho mot chiec xe 0.13 thi ca phong 10x10 thanh vung cam.

vx_max 0.5 -> 0.35: tran vat ly la MAX_WHEEL_RPM 120 voi banh 0.03225 m, tuc
0.405 m/s. De 0.5 thi Nav2 lap ke hoach theo toc do xe khong dat duoc.

Da kiem: xacro parse duoc ca sim:=true lan sim:=false, check_urdf hop le,
colcon build sach, firmware bien dich sach.

Co-Authored-By: Claude Opus 5 (1M context) <noreply@anthropic.com>

File: src/my_bot_description/description/gazebo_control.xacro (robot description, xacro)
@@ -5,6 +5,9 @@
             <left_joint>left_wheel_joint</left_joint>
             <right_joint>right_wheel_joint</right_joint>
-            <wheel_separation>1.1</wheel_separation>
-            <wheel_radius>0.05</wheel_radius>
+            <!-- PHAI khop robot.urdf.xacro va WHEEL_*_M trong firmware.
+                 Truoc day la 1.1 / 0.05 - so cua mot chiec xe duong kinh 1 m,
+                 khong dinh gi den xe that. -->
+            <wheel_separation>0.200</wheel_separation>
+            <wheel_radius>0.03225</wheel_radius>
             <max_linear_acceleration>1.0</max_linear_acceleration>
             <max_angular_acceleration>2.0</max_angular_acceleration>

File: src/my_bot_description/description/robot.urdf.xacro (robot description, xacro)
@@ -5,7 +5,35 @@
                      /scan va /odom do ESP32 phat, khong phai Gazebo. -->
     <xacro:arg name="sim" default="true" />
-    <xacro:if value="$(arg sim)">
-        <xacro:include filename="gazebo_control.xacro" />
-    </xacro:if>
+    <!-- ====================================================================
+         KICH THUOC XE
+         ====================================================================
+         Nhom 1 - DO BANG THUOC tren xe that. Sua o day la sua moi noi.
+         Ba file khac phai khop voi cac so nay, xem cuoi khoi nay. -->
+    <xacro:property name="wheel_separation" value="0.200"/>  <!-- tam - tam hai banh sau -->
+    <xacro:property name="wheel_radius"     value="0.03225"/><!-- duong kinh 64.5 mm -->
+    <xacro:property name="wheel_x"          value="-0.014"/> <!-- truc banh sau lui 14 mm sau tam -->
+    <xacro:property name="caster_x"         value="0.035"/>  <!-- banh da huong tien 35 mm truoc tam -->
+    <xacro:property name="body_radius"      value="0.0907"/> <!-- duong kinh than 181.40 mm -->
+    <!-- Nhom 2 - CHUA DO, dang la so dat tam cho hinh hoc dung duoc.
+         Sai cac so nay khong lam odometry sai, chi lam hinh trong RViz va
+         vat ly trong Gazebo khong giong that. Do roi thi sua vao day. -->
+    <xacro:property name="body_height"      value="0.040"/>  <!-- be day than xe -->
+    <xacro:property name="wheel_width"      value="0.026"/>  <!-- be rong lop -->
+    <xacro:property name="caster_radius"    value="0.015"/>  <!-- ban kinh bi da huong -->
+    <xacro:property name="lidar_z"          value="0.075"/>  <!-- tam LiDAR cao hon mat san -->
+    <xacro:property name="imu_z"            value="0.055"/>  <!-- tam BNO055 cao hon mat san -->
+    <xacro:property name="body_mass"        value="1.2"/>
+    <xacro:property name="wheel_mass"       value="0.05"/>
+    <xacro:property name="caster_mass"      value="0.02"/>
+    <!-- BA CHO KHAC PHAI KHOP VOI NHOM 1:
+           gazebo_control.xacro       <wheel_separation> va <wheel_radius>
+           firmware/.../esp32_agv_base.ino   WHEEL_SEPARATION_M, WHEEL_RADIUS_M
+           config/navigation.yaml     robot_radius (= diem xa tam nhat, xem duoi)
+         Diem xa tam nhat KHONG phai mep than xe (0.0907) ma la goc ngoai cua
+         banh sau, vi banh nho ra ngoai than:
+           x = wheel_x - wheel_radius = -0.014 - 0.03225 = -0.046
+           y = wheel_separation/2 + wheel_width/2 = 0.100 + 0.013 = 0.113
+           khoang cach = sqrt(0.046^2 + 0.113^2) = 0.122 m
+         -> navigation.yaml dat robot_radius 0.13 (co bien 8 mm). -->
     <material name="white"><color rgba="1 1 1 1" /></material>
     <material name="blue"><color rgba="0.2 0.2 1 1"/></material>
@@ -13,5 +41,6 @@
     <material name="orange"><color rgba="1 0.5 0 1"/></material>
     <material name="red"><color rgba="1 0 0 1"/></material>
-    <!-- Base Footprint (Required for Nav2 & SLAM) -->
+    <!-- base_footprint nam tren MAT SAN. base_link trung voi no, nen moi toa
+         do z duoi day deu la chieu cao so voi san. -->
     <link name="base_footprint"/>
     <joint name="base_footprint_joint" type="fixed">
@@ -27,37 +56,49 @@
     </joint>
     <link name="chassis">
-        <visual>
-            <origin xyz="0 0 0.075"/>
-            <geometry><cylinder radius="0.5" length="0.15"/></geometry>
+        <!-- Than dat o ngang tam truc banh -> gam cao 12 mm -->
+        <visual>
+            <origin xyz="0 0 ${wheel_radius}"/>
+            <geometry><cylinder radius="${body_radius}" length="${body_height}"/></geometry>
             <material name="orange"/>
         </visual>
         <collision>
-            <origin xyz="0 0 0.075"/>
-            <geometry><cylinder radius="0.5" length="0.15"/></geometry>
-        </collision>
-        <inertial>
-            <origin xyz="0 0 0.075" rpy="0 0 0"/>
-            <mass value="5.0"/>
-            <inertia ixx="0.321" ixy="0.0" ixz="0.0" iyy="0.321" iyz="0.0" izz="0.625"/>
-        </inertial>
-    </link>
+            <origin xyz="0 0 ${wheel_radius}"/>
+            <geometry><cylinder radius="${body_radius}" length="${body_height}"/></geometry>
+        </collision>
+        <inertial>
+            <origin xyz="0 0 ${wheel_radius}" rpy="0 0 0"/>
+            <mass value="${body_mass}"/>
+            <inertia
+                ixx="${body_mass*(3*body_radius*body_radius + body_height*body_height)/12}"
+                ixy="0.0" ixz="0.0"
+                iyy="${body_mass*(3*body_radius*body_radius + body_height*body_height)/12}"
+                iyz="0.0"
+                izz="${body_mass*body_radius*body_radius/2}"/>
+        </inertial>
+    </link>
+    <!-- Hai banh sau. Truc nam o z = wheel_radius thi lop vua cham san. -->
     <joint name="left_wheel_joint" type="continuous">
         <parent link="base_link"/>
         <child link="left_wheel"/>
-        <origin xyz="-0.1 0.55 0" rpy="-1.5707 0 0" />
+        <origin xyz="${wheel_x} ${wheel_separation/2} ${wheel_radius}" rpy="-1.5707 0 0"/>
         <axis xyz="0 0 1"/>
     </joint>
     <link name="left_wheel">
         <visual>
-            <geometry><cylinder radius="0.05" length="0.04"/></geometry>
+            <geometry><cylinder radius="${wheel_radius}" length="${wheel_width}"/></geometry>
             <material name="blue"/>
         </visual>
         <collision>
-            <geometry><cylinder radius="0.05" length="0.04"/></geometry>
+            <geometry><cylinder radius="${wheel_radius}" length="${wheel_width}"/></geometry>
         </collision>
         <inertial>
             <origin xyz="0 0 0" rpy="0 0 0"/>
-            <mass value="0.5"/>
-            <inertia ixx="0.000379" ixy="0.0" ixz="0.0" iyy="0.000379" iyz="0.0" izz="0.000625"/>
+            <mass value="${wheel_mass}"/>
+            <inertia
+                ixx="${wheel_mass*(3*wheel_radius*wheel_radius + wheel_width*wheel_width)/12}"
+                ixy="0.0" ixz="0.0"
+                iyy="${wheel_mass*(3*wheel_radius*wheel_radius + wheel_width*wheel_width)/12}"
+                iyz="0.0"
+                izz="${wheel_mass*wheel_radius*wheel_radius/2}"/>
         </inertial>
     </link>
@@ -65,40 +106,50 @@
         <parent link="base_link"/>
         <child link="right_wheel"/>
-        <origin xyz="-0.1 -0.55 0" rpy="1.5707 0 0" />
+        <origin xyz="${wheel_x} ${-wheel_separation/2} ${wheel_radius}" rpy="1.5707 0 0"/>
         <axis xyz="0 0 -1"/>
     </joint>
     <link name="right_wheel">
         <visual>
-            <geometry><cylinder radius="0.05" length="0.04"/></geometry>
+            <geometry><cylinder radius="${wheel_radius}" length="${wheel_width}"/></geometry>
             <material name="blue"/>
         </visual>
         <collision>
-            <geometry><cylinder radius="0.05" length="0.04"/></geometry>
+            <geometry><cylinder radius="${wheel_radius}" length="${wheel_width}"/></geometry>
         </collision>
         <inertial>
             <origin xyz="0 0 0" rpy="0 0 0"/>
-            <mass value="0.5"/>
-            <inertia ixx="0.000379" ixy="0.0" ixz="0.0" iyy="0.000379" iyz="0.0" izz="0.000625"/>
-        </inertial>
-    </link>
+            <mass value="${wheel_mass}"/>
+            <inertia
+                ixx="${wheel_mass*(3*wheel_radius*wheel_radius + wheel_width*wheel_width)/12}"
+                ixy="0.0" ixz="0.0"
+                iyy="${wheel_mass*(3*wheel_radius*wheel_radius + wheel_width*wheel_width)/12}"
+                iyz="0.0"
+                izz="${wheel_mass*wheel_radius*wheel_radius/2}"/>
+        </inertial>
+    </link>
+    <!-- Banh da huong phia truoc. Tam o z = caster_radius thi bi vua cham san. -->
     <joint name="front_caster_joint" type="fixed">
         <parent link="chassis"/>
         <child link="front_caster"/>
-        <origin xyz="0.4 0 0"/>
+        <origin xyz="${caster_x} 0 ${caster_radius}"/>
     </joint>
     <link name="front_caster">
         <visual>
-            <geometry><sphere radius="0.05"/></geometry>
+            <geometry><sphere radius="${caster_radius}"/></geometry>
             <material name="black"/>
         </visual>
         <collision>
-            <geometry><sphere radius="0.05"/></geometry>
+            <geometry><sphere radius="${caster_radius}"/></geometry>
         </collision>
         <inertial>
             <origin xyz="0 0 0" rpy="0 0 0"/>
-            <mass value="0.1"/>
-            <inertia ixx="0.0001" ixy="0.0" ixz="0.0" iyy="0.0001" iyz="0.0" izz="0.0001"/>
-        </inertial>
-    </link>
+            <mass value="${caster_mass}"/>
+            <inertia
+                ixx="${2*caster_mass*caster_radius*caster_radius/5}" ixy="0.0" ixz="0.0"
+                iyy="${2*caster_mass*caster_radius*caster_radius/5}" iyz="0.0"
+                izz="${2*caster_mass*caster_radius*caster_radius/5}"/>
+        </inertial>
+    </link>
+    <!-- Bi da huong khong duoc co ma sat, neu khong xe se khong quay not -->
     <gazebo reference="front_caster">
         <mu1>0.0</mu1>
@@ -109,9 +160,9 @@
         <parent link="chassis"/>
         <child link="lidar_link"/>
-        <origin xyz="0 0 0.17" rpy="0 0 0"/>
+        <origin xyz="0 0 ${lidar_z}" rpy="0 0 0"/>
     </joint>
     <link name="lidar_link">
         <visual>
-            <geometry><cylinder radius="0.05" length="0.04"/></geometry>
+            <geometry><cylinder radius="0.030" length="0.030"/></geometry>
             <material name="black"/>
         </visual>
@@ -144,10 +195,9 @@
     </xacro:if>
     <!-- IMU BNO055. Firmware phat /imu/data voi frame_id = imu_link,
-         neu thieu link nay TF se bao loi "frame does not exist".
-         SUA origin cho dung cho ban gan IMU tren xe that. -->
+         neu thieu link nay TF se bao loi "frame does not exist". -->
     <joint name="imu_joint" type="fixed">
         <parent link="chassis"/>
         <child link="imu_link"/>
-        <origin xyz="0 0 0.16" rpy="0 0 0"/>
+        <origin xyz="0 0 ${imu_z}" rpy="0 0 0"/>
     </joint>
     <link name="imu_link"/>
