Commit message: Firmware ESP32 hop nhat cho xe that + tach cau hinh sim/that
Gop 3 sketch Arduino thanh mot firmware duy nhat chay tren 1 con ESP32,
thay the hoan toan plugin DiffDrive va gpu_lidar cua Gazebo de Nav2 chay
tren xe that y het mo phong.

firmware/esp32_agv_base/esp32_agv_base.ino
- Nhan  /cmd_vel
- Phat  /scan /odom /tf (odom->base_footprint) /imu/data
- LiDAR giu nguyen tu ydlidar_microros.ino (ping-pong buffer, ngan sach MTU)
- PID + feedforward + bao ve sai chieu/ket banh lay tu motor_1_wheel_l298n.ino,
  nhan doi cho 2 banh. Dung he so ban L298N (Kf 1.8, deadband 30, PWM 5 kHz),
  KHONG phai ban BTS7960.
- Giu trinh tu ha ENA truoc khi lat IN1/IN2 de tranh soc dong qua cau H.
- Khung micro-ROS Wi-Fi + BNO055 lay tu Code-_xe_ros2.ino.
- Bo: bam line, 5 cam bien quang, lenh L/R/F/B, std_msgs/String, CLI Serial.
- Odometry tich phan Runge-Kutta bac 2, goc quay lay tu gyro (chinh xac hon
  encoder nhieu vi khong bi truot banh).
- Timeout /cmd_vel 500 ms va dung dong co truoc khi restart khi mat agent.
- Phan chia loi: Core 1 chi doc UART LiDAR; Core 0 chay motor_task (uu tien 3,
  50 Hz) va ros_task (uu tien 1).
- Chan GPIO chon lai de 3 sketch khong dam nhau, tranh chan flash va strapping.

Phia ROS
- robot.urdf.xacro: them arg sim (true/false) de bo plugin Gazebo khi chay xe
  that; them imu_link cho frame cua /imu/data.
- bringup_real.launch.py: micro_ros_agent + robot_state_publisher, thay cho
  gazebo.launch.py.
- navigation.launch.py: them arg use_sim_time.
- navigation.yaml: bo 8 dong use_sim_time. Nav2 Jazzy cap tham so nay bang
  SetParameter tu launch arg va KHONG ghi de qua param_rewrites, de lai trong
  yaml se thanh hai nguon su that.
- grid_navigator.py: use_sim_time khong con dong cung, chay xe that bang
  'python3 grid_navigator.py --real'.

Sua loi tranh chap luong trong grid_navigator.py
MultiThreadedExecutor cho phep costmap_callback va timer replan chay dong
thoi. Mot vat can kich hoat 4 luot huy/replan chong cheo, log hien dau thoi
gian dao nguoc. Them khoa trang thai va giu is_canceling cho toi khi Nav2
chap nhan goal moi. Chay lai kich ban: con dung 1 lan replan.

Co-Authored-By: Claude Opus 5 (1M context) <noreply@anthropic.com>

File: src/my_bot_description/description/robot.urdf.xacro (robot description, xacro)
@@ -1,5 +1,11 @@
 <?xml version="1.0"?>
 <robot xmlns:xacro="http://www.ros.org/wiki/xacro" name="my_bot">
-    <xacro:include filename="gazebo_control.xacro" />
+    <!-- sim=true  : nap plugin + sensor cua Gazebo (chay mo phong)
+         sim=false : chi con phan co khi thuan tuy, dung cho xe that vi luc do
+                     /scan va /odom do ESP32 phat, khong phai Gazebo. -->
+    <xacro:arg name="sim" default="true" />
+    <xacro:if value="$(arg sim)">
+        <xacro:include filename="gazebo_control.xacro" />
+    </xacro:if>
     <material name="white"><color rgba="1 1 1 1" /></material>
     <material name="blue"><color rgba="0.2 0.2 1 1"/></material>
@@ -111,4 +117,5 @@
         </visual>
     </link>
+    <xacro:if value="$(arg sim)">
     <gazebo reference="lidar_link">
         <sensor name="lidar" type="gpu_lidar">
@@ -135,3 +142,13 @@
         </sensor>
     </gazebo>
+    </xacro:if>
+    <!-- IMU BNO055. Firmware phat /imu/data voi frame_id = imu_link,
+         neu thieu link nay TF se bao loi "frame does not exist".
+         SUA origin cho dung cho ban gan IMU tren xe that. -->
+    <joint name="imu_joint" type="fixed">
+        <parent link="chassis"/>
+        <child link="imu_link"/>
+        <origin xyz="0 0 0.16" rpy="0 0 0"/>
+    </joint>
+    <link name="imu_link"/>
 </robot>

Commit message: mo hinh xe: wheel_width 26 mm da duoc do, chuyen sang nhom da do
Gia tri khong doi (dung bang so dat tam truoc do) nen hinh hoc va robot_radius
giu nguyen. Nhung gio ca ba so trong phep tinh robot_radius deu la so do that:
  sqrt(0.046^2 + 0.113^2) = 0.122 -> robot_radius 0.13

Co-Authored-By: Claude Opus 5 (1M context) <noreply@anthropic.com>

File: src/my_bot_description/description/robot.urdf.xacro (robot description, xacro)
@@ -15,9 +15,9 @@
     <xacro:property name="caster_x"         value="0.035"/>  <!-- banh da huong tien 35 mm truoc tam -->
     <xacro:property name="body_radius"      value="0.0907"/> <!-- duong kinh than 181.40 mm -->
+    <xacro:property name="wheel_width"      value="0.026"/>  <!-- be rong lop 26 mm -->
     <!-- Nhom 2 - CHUA DO, dang la so dat tam cho hinh hoc dung duoc.
          Sai cac so nay khong lam odometry sai, chi lam hinh trong RViz va
          vat ly trong Gazebo khong giong that. Do roi thi sua vao day. -->
     <xacro:property name="body_height"      value="0.040"/>  <!-- be day than xe -->
-    <xacro:property name="wheel_width"      value="0.026"/>  <!-- be rong lop -->
     <xacro:property name="caster_radius"    value="0.015"/>  <!-- ban kinh bi da huong -->
     <xacro:property name="lidar_z"          value="0.075"/>  <!-- tam LiDAR cao hon mat san -->
@@ -31,9 +31,10 @@
            config/navigation.yaml     robot_radius (= diem xa tam nhat, xem duoi)
          Diem xa tam nhat KHONG phai mep than xe (0.0907) ma la goc ngoai cua
-         banh sau, vi banh nho ra ngoai than:
+         banh sau, vi hai banh cach nhau 200 mm trong khi than chi rong 181.40:
            x = wheel_x - wheel_radius = -0.014 - 0.03225 = -0.046
            y = wheel_separation/2 + wheel_width/2 = 0.100 + 0.013 = 0.113
            khoang cach = sqrt(0.046^2 + 0.113^2) = 0.122 m
-         -> navigation.yaml dat robot_radius 0.13 (co bien 8 mm). -->
+         Ca ba so trong phep tinh nay deu do that -> navigation.yaml dat
+         robot_radius 0.13 (co bien 8 mm). -->
     <material name="white"><color rgba="1 1 1 1" /></material>
     <material name="blue"><color rgba="0.2 0.2 1 1"/></material>

Commit message: URDF: base_footprint tai tam truc banh; dich la o dang dung - chay toi neu o o phia truoc
- robot.urdf.xacro: base_footprint duoi truc banh (base_link truoc 14 mm). Truoc day
  xoay tai cho 180 do lam vi tri xe troi 2.8 cm ma odometry khong biet (2 xe that:
  lech dich 3-4.4 cm sau cu xoay cuoi).
- grid_navigator/fleet_agent stay_put(): o nam truoc mui (<= 30 do) -> chay thang toi
  (Nav2 dung som 8 cm vi vat can thoang qua); ben hong/sau lung va <= 10 cm -> bo qua.
- Thu that 2 xe: 6 buoc deu dung logic mo phong, khong va (min 59-60 cm).

Co-Authored-By: Claude Opus 5.5 <noreply@anthropic.com>

File: src/my_bot_description/description/robot.urdf.xacro (robot description, xacro)
@@ -42,11 +42,16 @@
     <material name="orange"><color rgba="1 0.5 0 1"/></material>
     <material name="red"><color rgba="1 0 0 1"/></material>
-    <!-- base_footprint nam tren MAT SAN. base_link trung voi no, nen moi toa
-         do z duoi day deu la chieu cao so voi san. -->
+    <!-- base_footprint nam tren MAT SAN, ngay duoi TAM TRUC BANH (tam xoay cua xe
+         vi sai). base_link = tam than, truoc truc 14 mm (-wheel_x); moi toa do
+         z duoi day deu la chieu cao so voi san.
+         Truoc 2026-10-10 base_footprint o tam THAN: xoay tai cho 180 do lam "vi tri
+         xe" (odom/AMCL/sa ban) troi 2.8 cm (90 do: 2 cm) ma odometry vi sai khong
+         biet -> xe 2 xe that toi dich lech 3-4.4 cm sau cu xoay cuoi. Gio xoay tai
+         cho khong doi vi tri; tam than luon nam truoc nut 1.4 cm theo mui xe. -->
     <link name="base_footprint"/>
     <joint name="base_footprint_joint" type="fixed">
         <parent link="base_footprint"/>
         <child link="base_link"/>
-        <origin xyz="0 0 0" rpy="0 0 0"/>
+        <origin xyz="${-wheel_x} 0 0" rpy="0 0 0"/>
     </joint>
     <link name="base_link"></link>
